File: hardware/tkmem128.kicad_sch (KiCad schematic)
At the start: 24 parts, among them J1 Para a expansora, U1 GAL20V8B, U2 74HCT273, U3 AS6C1008-55PCN, U4 27C256

Commit message: Esquematicos e silk rearranjados; pendencia do plano do soquete de borda
Esquematico das duas placas redesenhado a mao (havia simbolos saindo da
folha e sinais misturados) e serigrafia reorganizada. Conferido: ERC 0,
DRC 0, e a netlist exportada bate no a no com a intencao de projeto nas
duas placas (74 e 53 nets, zero divergencia).

Os geradores em tools/ passam a ser ferramenta de bootstrap: gen_schematic.py
e gen_pcb.py sobrescreveriam o ajuste manual. A fonte corrente e o conteudo
de hardware/. Documentado no README de tools/.

Registrada uma pendencia real da placa expansora (item 1b de
docs/ANTES-DE-FABRICAR.md): nas placas originais a fenda do soquete que
recebe os dedos do TK fica NO PLANO da placa, alinhada com os dedos de
passagem. O footprint atual e uma grade 2x28 de furos comuns, ou seja, o
conector monta por cima e a fenda fica alguns milimetros acima do plano —
o que joga a expansora abaixo do plano do TK e faz o periferico seguinte da
corrente descer outro tanto. Falta medir o conector para decidir entre
straddle mount e montagem por baixo.

Saidas de fabricacao e renders regerados a partir dos arquivos revisados.

Co-Authored-By: Claude Opus 5 <noreply@anthropic.com>
Other:
- moved on the sheet: C1, C2, C3, C4, C5, C6, D1, J1, JP1, JP2, JP3, JP4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

Commit message: Principal: trilha 0,50 mm, reposicionada para rotear
Voce estava certo nos dois pontos. Medindo o que estava la: dos 96 vaos entre
ilhas vizinhas de DIP, 10 tinham 2 ou 3 trilhas passando. E a ilha LongPads
deixa 0,94 mm de vao, onde cabe EXATAMENTE UMA trilha em qualquer largura
sensata — 0,25/0,15 precisava de 0,95 mm para duas. O autorouter espremeu onde
nao cabia.

REGRAS      sinal 0,25 -> 0,50 mm | alimentacao 0,60 -> 1,00 | isolacao 0,14 ->
            0,20. Com isso o canal duplo entre ilhas fica proibido por
            construcao, e nao por sorte.

POSICIONAMENTO. O arranjo velho tinha DUAS fileiras de passivos atravessando a
placa de lado a lado (C1..C6+D1+TP em y=47,2; R2..SJ2 em y=53,3), bem entre o
conector e os CIs — por onde passam A0..A13 e D0..D7. E os cinco capacitores de
desacoplamento ficavam a 40 mm dos pinos que deveriam desacoplar.

Os quatro CIs tambem estavam VERTICAIS: os 16 pinos de um lado empilhados numa
reta de 38 mm, obrigando todo sinal vindo do conector a subir por um canal
estreito ao lado do CI e depois virar. Girados para HORIZONTAL, a fileira de
pinos fica paralela ao conector e cada sinal sobe quase reto — e o que a placa
Luccas faz, e e por isso que as trilhas dela podem ser gordas.

  y  4..22   U4 EPROM (horizontal)     |  JP1..JP4, R2..R5, D1, TP1, TP2
  y 27..45   U3 SRAM  (horizontal)     |  U1 GAL / U2 74HCT273
  y 48..57   corredor limpo de ponta a ponta
  y 60..65   conector

Cada capacitor de desacoplamento foi para junto do pino de +5V do seu CI.

SJ1 E SJ2 SAIRAM (sua sugestao, e estava certa). Eram terra extra OPCIONAL em
pinos que so sao GND numa das maquinas — 7 no ZX Spectrum, 15 no TK — e a
propria documentacao ja mandava deixar os dois abertos. Em troca, cada um puxava
uma rede do conector ate o outro extremo da placa. Sozinha essa remocao nao
fechou as ultimas nets, mas simplificou a placa e eliminou uma colisao de
contorno com C5. Quem quiser o terra extra solda um fio do pino ao plano.

BUG NO PIPELINE, ach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
Parts:
- removed SJ1: GND pino 7, Jumper:SolderJumper-2_P1.3mm_Open_RoundedPad1.0x1.5mm, symbol Jumper:SolderJumper_2_Open
- removed SJ2: GND pino 15, Jumper:SolderJumper-2_P1.3mm_Open_RoundedPad1.0x1.5mm, symbol Jumper:SolderJumper_2_Open
Connections:
- net BUS_P07: no longer names the net of J1.7 (NC/GND_(7))
- net BUS_P15: no longer names the net of J1.15 (GND/NC_(15))
- no-connect marks 0 -> 2
