File: hardware/tkmem128.kicad_sch (KiCad schematic)
At the start: 22 parts, among them J1 Para a expansora, U1 GAL20V8B, U2 74HCT273, U3 AS6C1008-55PCN, U4 27C256

Commit message: Auto-desativacao vai para o pino 29; JP4 deixa de existir
Sua pesquisa resolve o pior risco que sobrava no projeto. Conferi antes de mexer,
porque errar isso custa o micro de quem monta:

  Pinagem oficial do TK, arquivada em docs/ (imagem, extraida do PDF do Luccas):
  o pino 29 esta marcado **N.C.**  E nas fotos do cartao do TK o dedo 29, como o
  17, nao tem trilha nenhuma chegando.

  O lado do Spectrum (28A livre) e a sua pesquisa. Vale registrar que o busdef
  deste projeto sinaliza TODO pino que difere entre as duas maquinas — 16/17/18
  como Y/V/U do video, 34/35/37 como alimentacao divergente — e o 29 nunca teve
  ressalva nenhuma. Duas fontes independentes concordando.

Com o pino 29 sendo N.C. nas DUAS maquinas, o pull-up pode ser PERMANENTE: num
Spectrum nao ha nada ligado ali, num TK ele faz o que tem que fazer. Entao:

  JP4 SAIU. Com ele saiu o aviso "NUNCA feche JP4 em ZX Spectrum" da serigrafia,
  do README, do MONTAGEM e do PREPARAR-O-TK. Nao existe mais posicao errada para
  escolher — o risco nao foi mitigado, foi eliminado.

R4 fica, e continua em 1k: e o limite de corrente, e nao monta-lo libera o pino
29 para quem precisar dele. Conferi que 1k basta: a placa Luccas original usava
10k nesse mesmo ponto e funcionava, o que prova que o pino 10 do IC27 e entrada
livre, sem nada disputando.

UM DETALHE PRATICO que a documentacao agora avisa: o pino 29 esta na fileira de
CIMA (29..56), na face do cartao do TK oposta a dos pinos 1..28. Quem seguir as
fotos da modificacao original vai soldar do outro lado da placa-mae.

REROTEAMENTO. A mudanca de pino move a rede para o canto oposto da placa, entao a
principal foi reroteada inteira. O Freerouting fechou 73 das 74 e deixou A14 —
que nao era a rede alterada, e a diferenca de 1 net entrou no ruido do
determinismo dele. Fiz A14 a mao pela margem direita, com um detalhe medido: a
janela entre a ilha do GAL (que acaba em x=77,44) e a folga de borda tem 0,30 mm
de largura, e a trilha de 0,5 mm cabe centrada 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
Parts:
- removed JP4: AUTO-DESATIVA 32K, Connector_PinHeader_2.54mm:PinHeader_1x02_P2.54mm_Vertical, symbol Connector_Generic:Conn_01x02
Connections:
- net BUS_P29 is gone; now on net RAMDIS: J1.29 (NC_(29))
- net RAMDIS_DRV is gone; now on net RAMDIS: R4.2
- net RAMDIS: no longer J1.17 (RAMDIS_(17))
- new net BUS_P17: J1.17 (RAMDIS_(17))
Changed lines of the file:
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@@
 	(wire
 		(pts
-			(xy 496.57 279.4) (xy 492.76 279.4)
-		)
-		(stroke
-			(width 0)
-			(type default)
-		)
-	)
-	(wire
-		(pts
 			(xy 307.34 116.84) (xy 303.53 116.84)
 		)
@@
 		)
 	)
-	(wire
-		(pts
-			(xy 496.57 276.86) (xy 492.76 276.86)
-		)
-		(stroke
-			(width 0)
-			(type default)
-		)
-	)
 	(global_label "GND"
 		(shape bidirectional)
@@
 		)
 	)
-	(global_label "RAMDIS"
+	(global_label "BUS_P17"
 		(shape bidirectional)
 		(at 46.99 196.85 180)
@@
 		)
 	)
-	(global_label "RAMDIS"
-		(shape bidirectional)
-		(at 492.76 279.4 180)
-		(fields_autoplaced yes)
-		(effects
-			(font
-				(size 1.27 1.27)
-			)
-			(justify right)
-		)
-		(property "Intersheetrefs" "${INTERSHEET_REFS}"
-			(at 492.76 279.4 0)
-			(hide yes)
-			(show_name no)
-			(do_not_autoplace no)
-			(effects
-				(font
-					(size 1.27 1.27)
-				)
-			)
-		)
-	)
 	(global_label "D4"
 		(shape bidirectional)
@@
 		)
 	)
-	(global_label "BUS_P29"
+	(global_label "RAMDIS"
 		(shape bidirectional)
 		(at 105.41 224.79 0)
@@
 		)
 	)
-	(global_label "RAMDIS_DRV"
+	(global_label "RAMDIS"
 		(shape bidirectional)
 		(at 521.97 96.52 90)
@@
 		)
 	)
-	(global_label "RAMDIS_DRV"
-		(shape bidirectional)
-		(at 492.76 276.86 180)
-		(fields_autoplaced yes)
-		(effects
-			(font
-				(size 1.27 1.27)
-			)
-			(justify right)
-		)
-		(property "Intersheetrefs" "${INTERSHEET_REFS}"
-			(at 492.76 276.86 0)
-			(hide yes)
-			(show_name no)
-			(do_not_autoplace no)
-			(effects
-				(font
-					(size 1.27 1.27)
-				)
-			)
-		)
-	)
 	(global_label "A7"
 		(shape bidirectional)
@@
 					(unit 1)
 				)
-			)
-		)
-	)
-	(symbol
-		(lib_id "Connector_Generic:Conn_01x02")
-		(at 501.65 276.86 0)
-		(unit 1)
-		(body_style 1)
-		(exclude_from_sim no)
-		(in_bom yes)
-		(on_board yes)
-		(in_pos_files yes)
-		(dnp no)
-		(property "Reference" "JP4"
-			(at 501.65 271.78 0)
-			(show_name no)
-			(do_not_autoplace no)
-			(effects
-				(font
-					(size 1.27 1.27)
-				)
-				(justify left)
-			)
-		)
-		(property "Value" "AUTO-DESATIVA 32K"
-			(at 501.65 274.32 0)
-			(show_name no)
-			(do_not_autoplace no)
-			(effects
-				(font
-					(size 1.27 1.27)
-				)
-				(justify left)
-			)
-		)
-		(property "Footprint" "Connector_PinHeader_2.54mm:PinHeader_1x02_P2.54mm_Vertical"
-			(at 501.65 276.86 0)
-			(hide yes)
-			(show_name no)
-			(do_not_autoplace no)
-			(effects
-				(font
-					(size 1.27 1.27)
-				)
-			)
-		)
-		(property "Datasheet" ""
-			(at 501.65 276.86 0)
-			(hide yes)
-			(show_name no)
-			(do_not_autoplace no)
-			(effects
-				(font
-					(size 1.27 1.27)
-				)
-			)
-		)
-		(property "Description" "Fechado = injeta nivel 1 no pino 17 e desliga a RAM interna do TK. NAO fechar em ZX Spectrum: la o pino 17 e o V do video componente"
-			(at 501.65 276.86 0)
-			(hide yes)
-			(show_name no)
-			(do_not_autoplace no)
-			(effects
-				(font
-					(size 1.27 1.27)
-				)
-			)
-		)
-		(pin "1"
-		)
-		(pin "2"
-		)
-		(instances
-			(project "tkmem128"
-				(path "/214ef319-1120-feeb-674c-ee15bc976f0e"
-					(reference "JP4")
-					(unit 1)
-				)
