File: hardware/tkmem128-ii.kicad_pcb (KiCad board)
At the start: 4 copper layers, 78.7 x 66 mm, 22 parts, among them J1 Barramento TK, U1 GAL20V8B, U2 74HCT273, U3 AS6C1008-55PCN, U4 27C256

Commit message: Poda os desvios que o Freerouting deixou: 54,7 mm em 41 cadeias
O `ROMA14` que o Leonardo apontou subia por cima de uma ilha do R5,
atravessava, e descia pelo vao de 1,27 mm ENTRE as duas ilhas do R5 — com
0,22 mm de folga de cada lado — so para voltar a mesma altura de onde tinha
saido. Reto por baixo cabia, e com MAIS folga (0,25). Nao era restricao: era
resto de uma iteracao anterior do autoroteador, que roteia e depois otimiza mas
nao desfaz escadinha.

`tools/endireita_trilhas.py` generaliza o teste que fiz a mao naquele caso.
Quebra cada rede em cadeias entre nos fixos (ilha, via, bifurcacao) e tenta
trocar o pedaco entre dois vertices por um caminho no estilo da placa — um
trecho reto ou dois em "L" com canto de 45. Cada candidato e medido ponto a
ponto, a cada 0,02 mm, contra todo o cobre daquela face que nao seja da mesma
rede, mais a margem e a area de exclusao do furo. So entra se couber e encurtar.
Nao muda de camada, nao mexe em via, nao muda as pontas: e poda local.

Resultado, rodando ate convergir (cada passada muda a decomposicao em cadeias e
abre a seguinte):

    F.Cu  1546,4 -> 1503,6 mm
    B.Cu  1524,5 -> 1511,6 mm
    cantos de 90 graus  23 -> 0

Duas coisas que a primeira leitura da lista sugeria erro e nao eram:

- o `A14` aparecia com -13,51 mm, o que parecia corte de caminho. Nao e: ele
  chanfrou os dois cantos de 90 graus da volta pela margem. Continua rente a
  margem, so com 45 nas quinas.
- vinte entradas com exatamente -1,00 mm. E aritmetica, nao bug: sao cantos de
  90 com pernas de 1,70 mm, a saida padrao de uma ilha de DIP, e
  1,70+1,70-1,70*raiz(2) = 1,00.

O unico canto de 90 que sobrou no relatorio nao e canto: e a via de A11 em
(3,245 ; 38,715), onde tres ramos se encontram. Ponto fixo por definicao.

DRC 0/0, ERC 0, os quatro conferidores OK.

Co-Authored-By: Claude Opus 5 <noreply@anthropic.com>
Routing:
- net A14: track 52.1 -> 38.6 mm
- net ROMA14: track 96.5 -> 92.3 mm
- net SA15: track 77.6 -> 75.6 mm
- net A1: track 88.8 -> 86.8 mm
- net RAMCS_N: track 36.3 -> 34.3 mm
- net D2: track 64.6 -> 62.7 mm
- net SA14: track 55.9 -> 53.9 mm
- net BANK4: track 19.7 -> 17.7 mm
- net SA16: track 62.3 -> 60.3 mm
- net D0: track 66.1 -> 64.1 mm
- net A11: track 100.3 -> 98.3 mm
- net D1: track 64.4 -> 62.4 mm
- net WR_N: track 78.2 -> 76.3 mm
- net D7: track 85.6 -> 83.8 mm
- net A13: track 111.6 -> 110.2 mm
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