File: hardware/tkmem128-ii.kicad_sch (KiCad schematic)
At the start: 21 parts, among them J1 Para a expansora, U1 GAL20V8B, U2 74HCT273, U3 AS6C1008-55PCN, U4 27C256

Commit message: Corrige o nome do projeto onde ele fica impresso
A renomeacao para TKMEM-128 II passou por cima do bloco de titulo dos dois
esquematicos, que sai no PDF entregue em production/, e do cabecalho do .jed,
que sai na tela de quem grava a GAL. Os dois ainda diziam "TKMEM-128 KiCad",
e o .jed ainda apontava para github.com/lrrosa/tkmem128-kicad.

De quebra, o esquematico da tira carregava o titulo da placa PRINCIPAL — veio
junto quando o projeto foi copiado. Agora diz o que ele e.

O .jed foi regerado por galgen.py so pelo cabecalho: antes de escrever, as
equacoes foram reconstruidas e comparadas fusivel a fusivel com o arquivo
antigo (0 divergencias em 2706) e o resultado reconferido contra o
GAL20V8B.JED do acervo — 0 divergencias, checksum 5752 nos tres.

Os geradores em tools/ tambem foram corrigidos para nao reintroduzir o nome
velho, e producao.sh regerou gerbers, PDF, BOM, posicoes, renders e zips.
confere_saidas / _compatibilidade / _alinhamento / _svg: todos OK.

Co-Authored-By: Claude Opus 5 <noreply@anthropic.com>
Other:
- title: TKMEM-128 KiCad - expansao de 128K para TK90X/TK95 -> TKMEM-128 II - expansao de 128K para TK90X/TK95
Changed lines of the file:
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@@
 	(paper "A2")
 	(title_block
-		(title "TKMEM-128 KiCad - expansao de 128K para TK90X/TK95")
+		(title "TKMEM-128 II - expansao de 128K para TK90X/TK95")
 		(rev "1.0")
 		(company "Derivado de Velesoft (2009) e Luccas Eletronica (2012) - CERN-OHL-S v2")

Commit message: Legenda diz ZX Spectrum 48K e clones — e o pino 17 parou de mentir
O bloco de titulo dos dois esquematicos dizia "para TK90X/TK95". Errado desde
que a placa voltou a servir no ZX Spectrum 48K: o circuito e do Velesoft e
nasceu para o Spectrum, os TKs e que sao os clones. Agora diz "ZX Spectrum 48K
e clones", e o mesmo vale para o titulo em netlist.py/netlist_exp.py e para as
descricoes de simbolo e footprint.

De quebra, a mesma afirmacao errada estava na SERIGRAFIA da tira, em F.SilkS —
essa sai impressa na placa. Virou "ZX SPECTRUM 48K E CLONES".

Os `tags`/`ki_keywords` continuam citando TK90X e TK95 de proposito: ali listar
as duas familias e justamente o que se quer, sao palavras de busca.

O QUE APARECEU AO REGERAR A BIBLIOTECA. O simbolo do conector ainda rotulava
**pino 17 = RAMDIS e pino 29 = NC** — a pinagem de ANTES de mover a
auto-desativacao da RAM para o pino 29 por causa do video componente do
Spectrum. E tinha chegado aos dois esquematicos: o PDF entregue desenhava
exatamente a ligacao que fomos evitar, com o rotulo do pino contradizendo o
fio ligado nele (o global label ja dizia BUS_P17). Quatro rotulos por
esquematico: 16, 17, 18 e 29.

E a terceira vez que uma copia envelhece em silencio aqui — antes foram a ilha
do conector (biblioteca com 1,75 enquanto a placa usava 1,50) e o titulo do
bloco de legenda. Entao virou conferidor: `tools/confere_pinos.py` compara os
rotulos dos dois esquematicos e da biblioteca contra busdef.py, que e a fonte
unica da pinagem. Conferido com teste negativo nos dois formatos.

Detalhe que quase deixou o conferidor inutil: o gerador escreve "ROTULO (nn)"
com espaco, e e assim que fica no .kicad_sym, mas o KiCad troca por underscore
ao salvar um .kicad_sch. A primeira versao do padrao so aceitava underscore,
lia ZERO pino na biblioteca e passava "sem divergencia".

DRC 0/0 na principal, 0 violacoes na tira, ERC 0, os cinco conferidores OK.

Co-Authored-By: Claude Opus 5 <noreply@anthropic.com>
Other:
- title: TKMEM-128 II - expansao de 128K para TK90X/TK95 -> TKMEM-128 II - expansao de 128K para ZX Spectrum 48K e clones
Changed lines of the file:
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@@
 	(paper "A2")
 	(title_block
-		(title "TKMEM-128 II - expansao de 128K para TK90X/TK95")
+		(title "TKMEM-128 II - expansao de 128K para ZX Spectrum 48K e clones")
 		(rev "1.0")
 		(company "Derivado de Velesoft (2009) e Luccas Eletronica (2012) - CERN-OHL-S v2")

Commit message: Sincroniza J1 com o PCB na BOM e acrescenta a PALCE20V8H
A BOM sai do esquematico e as posicoes saem do PCB, e os dois discordavam
sobre J1: a BOM trazia o header 2x28 do prototipo descartado ("Para a
expansora", ZX_TK_Bus_Header_2x28) enquanto a placa ja tinha o conector de
borda TE 5645235 (ZX_TK_Bus_Socket_56). O tools/netlist.py ja estava
corrigido; so o .kicad_sch nunca foi ressincronizado, porque rodar o
gen_schematic.py apagaria o rearranjo manual do esquematico.

Como "Para a expansora" era o campo Value, o nome errado tambem saia
impresso ao lado de J1 no PDF do esquematico entregue.

A BOM da tira de expansao ja estava correta (ilhas de solda + dedos, sem
conector nenhum).

PALCE20V8H entra como terceira peca compativel em U1. Conferido antes de
afirmar: o .jed e QF2706/C5752 em modo complex (SYN=1, AC0=1, todas as
saidas combinatorias em tristate, nenhum registrador usado -- o latch e o
74HCT273 externo), que e a emulacao de um PAL20L8, justamente o que a
PALCE20V8H faz nativamente. Documentadas as duas ressalvas: selecionar o
dispositivo certo no programador (o mapa de fusiveis e igual, o algoritmo
de gravacao nao) e evitar os grades -5/-7, que consomem bem mais.

De quebra, apagado o footprint orfao ZX_TK_Bus_Header_2x28.kicad_mod e a
gen_header() que o gerava: nenhuma das duas placas o usava, e era ele que
sustentava a entrada errada na BOM. Conferido rodando o gerador num
diretorio temporario -- os 6 footprints restantes saem byte a byte
identicos aos da biblioteca.

ERC 0, DRC 0 nas duas placas. Nos gerbers mudou so o carimbo de data; a
geometria e identica.

Co-Authored-By: Claude Opus 5 <noreply@anthropic.com>
Parts:
- J1: value Para a expansora -> Barramento TK; footprint tkmem128:ZX_TK_Bus_Header_2x28 -> tkmem128:ZX_TK_Bus_Socket_56
Changed lines of the file:
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@@
 			)
 		)
-		(property "Value" "Para a expansora"
+		(property "Value" "Barramento TK"
 			(at 76.2 151.892 0)
 			(show_name no)
@@
 			)
 		)
-		(property "Footprint" "tkmem128:ZX_TK_Bus_Header_2x28"
+		(property "Footprint" "tkmem128:ZX_TK_Bus_Socket_56"
 			(at 76.2 191.77 0)
 			(hide yes)
@@
 			)
 		)
-		(property "Description" "Soquete femea 2x28 angular - liga a placa expansora"
+		(property "Description" "Conector de borda TE 5645235 soldado nesta placa. O corpo fica do lado OPOSTO aos componentes; os terminais atravessam e recebem a tira de expansao pelo lado dos componentes."
 			(at 76.2 191.77 0)
 			(hide yes)
@@
 			)
 		)
-		(property "Description" "Decodificador de enderecos (GAL20V8B ou ATF20V8B)"
+		(property "Description" "Decodificador de enderecos (GAL20V8B, ATF20V8B ou PALCE20V8H)"
 			(at 199.39 107.95 0)
 			(hide yes)
