File: hardware/expansor/tkmem128-ii-expansor.kicad_sch (KiCad schematic)
At the start: 2 parts, among them J1 Terminais do conector, J2 Passagem

Commit message: Corrige o nome do projeto onde ele fica impresso
A renomeacao para TKMEM-128 II passou por cima do bloco de titulo dos dois
esquematicos, que sai no PDF entregue em production/, e do cabecalho do .jed,
que sai na tela de quem grava a GAL. Os dois ainda diziam "TKMEM-128 KiCad",
e o .jed ainda apontava para github.com/lrrosa/tkmem128-kicad.

De quebra, o esquematico da tira carregava o titulo da placa PRINCIPAL — veio
junto quando o projeto foi copiado. Agora diz o que ele e.

O .jed foi regerado por galgen.py so pelo cabecalho: antes de escrever, as
equacoes foram reconstruidas e comparadas fusivel a fusivel com o arquivo
antigo (0 divergencias em 2706) e o resultado reconferido contra o
GAL20V8B.JED do acervo — 0 divergencias, checksum 5752 nos tres.

Os geradores em tools/ tambem foram corrigidos para nao reintroduzir o nome
velho, e producao.sh regerou gerbers, PDF, BOM, posicoes, renders e zips.
confere_saidas / _compatibilidade / _alinhamento / _svg: todos OK.

Co-Authored-By: Claude Opus 5 <noreply@anthropic.com>
Other:
- title: TKMEM-128 KiCad - expansao de 128K para TK90X/TK95 -> TKMEM-128 II - tira de expansao do barramento TK90X/TK95
Changed lines of the file:
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@@
 	(paper "A2")
 	(title_block
-		(title "TKMEM-128 KiCad - expansao de 128K para TK90X/TK95")
+		(title "TKMEM-128 II - tira de expansao do barramento TK90X/TK95")
 		(rev "1.0")
 		(company "Derivado de Velesoft (2009) e Luccas Eletronica (2012) - CERN-OHL-S v2")

Commit message: Legenda diz ZX Spectrum 48K e clones — e o pino 17 parou de mentir
O bloco de titulo dos dois esquematicos dizia "para TK90X/TK95". Errado desde
que a placa voltou a servir no ZX Spectrum 48K: o circuito e do Velesoft e
nasceu para o Spectrum, os TKs e que sao os clones. Agora diz "ZX Spectrum 48K
e clones", e o mesmo vale para o titulo em netlist.py/netlist_exp.py e para as
descricoes de simbolo e footprint.

De quebra, a mesma afirmacao errada estava na SERIGRAFIA da tira, em F.SilkS —
essa sai impressa na placa. Virou "ZX SPECTRUM 48K E CLONES".

Os `tags`/`ki_keywords` continuam citando TK90X e TK95 de proposito: ali listar
as duas familias e justamente o que se quer, sao palavras de busca.

O QUE APARECEU AO REGERAR A BIBLIOTECA. O simbolo do conector ainda rotulava
**pino 17 = RAMDIS e pino 29 = NC** — a pinagem de ANTES de mover a
auto-desativacao da RAM para o pino 29 por causa do video componente do
Spectrum. E tinha chegado aos dois esquematicos: o PDF entregue desenhava
exatamente a ligacao que fomos evitar, com o rotulo do pino contradizendo o
fio ligado nele (o global label ja dizia BUS_P17). Quatro rotulos por
esquematico: 16, 17, 18 e 29.

E a terceira vez que uma copia envelhece em silencio aqui — antes foram a ilha
do conector (biblioteca com 1,75 enquanto a placa usava 1,50) e o titulo do
bloco de legenda. Entao virou conferidor: `tools/confere_pinos.py` compara os
rotulos dos dois esquematicos e da biblioteca contra busdef.py, que e a fonte
unica da pinagem. Conferido com teste negativo nos dois formatos.

Detalhe que quase deixou o conferidor inutil: o gerador escreve "ROTULO (nn)"
com espaco, e e assim que fica no .kicad_sym, mas o KiCad troca por underscore
ao salvar um .kicad_sch. A primeira versao do padrao so aceitava underscore,
lia ZERO pino na biblioteca e passava "sem divergencia".

DRC 0/0 na principal, 0 violacoes na tira, ERC 0, os cinco conferidores OK.

Co-Authored-By: Claude Opus 5 <noreply@anthropic.com>
Other:
- title: TKMEM-128 II - tira de expansao do barramento TK90X/TK95 -> TKMEM-128 II - tira de expansao do barramento do ZX Spectrum 48K e clones
Changed lines of the file:
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@@
 	(paper "A2")
 	(title_block
-		(title "TKMEM-128 II - tira de expansao do barramento TK90X/TK95")
+		(title "TKMEM-128 II - tira de expansao do barramento do ZX Spectrum 48K e clones")
 		(rev "1.0")
 		(company "Derivado de Velesoft (2009) e Luccas Eletronica (2012) - CERN-OHL-S v2")
